File: chatmixv2.kicad_sch (KiCad schematic)
At the start: 29 parts, among them J1 USB_C_Receptacle_USB2.0_16P, J3 JTAG/SWD - MIPI-10, SW1 Mute, SW2 Mode, U1 STM32F072RBTx, U2 AP2112K-3.3, U3 LM393, U5 USBLC6-2SC6

Commit message: seperated connections with plugs
Parts:
- removed C10: 100 uF, symbol Device:C_US
- removed R3, R4: 1K, symbol Device:R_US
- removed U3: LM393, symbol Comparator:LM393
- added C13: 100nF, symbol Device:C_Small_US
- added J3C: Conn Mute, symbol Connector:Conn_01x02_Socket
- added J3P: Pin Mute, symbol Connector:Conn_01x02_Pin
- added J4C: Conn Mode, symbol Connector:Conn_01x02_Socket
- added J4P: Pin Mode, symbol Connector:Conn_01x02_Pin
- added J5C: Conn Pot, symbol Connector:Conn_01x03_Socket
- added J5P: Pin Pot, symbol Connector:Conn_01x03_Pin
- R8: value 4.7k -> 1k
- renumbered J3 to J2
Connections:
- net 3.3V: now also J5C.1 (Pin_1); no longer R8.1, RV1.1
- net GND: now also C13.2, J3C.2 (Pin_2), J4C.2 (Pin_2), J5C.3 (Pin_3); no longer RV1.3, SW1.1, SW1.3, SW2.1, SW2.3
- net at U1.8 (PC0): now also R8.2, C13.1; no longer RV1.2
- net at SW2.2, SW2.4: now also J4P.1 (Pin_1); no longer C12.1, U1.11 (PC3)
- net at SW1.2, SW1.4: now also J3P.1 (Pin_1); no longer C11.1, U1.10 (PC2)
- net at U1.9 (PC1): now also C11.1, J3C.1 (Pin_1); no longer R8.2
- new net: C12.1, J4C.1 (Pin_1), U1.10 (PC2)
- new net: J4P.2 (Pin_2), SW2.1, SW2.3
- new net: J5C.2 (Pin_2), R8.1
- new net: J3P.2 (Pin_2), SW1.1, SW1.3
- new net: J5P.1 (Pin_1), RV1.1
- new net: J5P.2 (Pin_2), RV1.2
- new net: J5P.3 (Pin_3), RV1.3
Other:
- moved on the sheet: C11, C12, R6, R7, R8, RV1, SW1, SW2

Commit message: added firmware stuff, usb descriptor for test board
Parts:
- added D1, D2, D3: PESD5V0L1UL, Diode_SMD:D_SOD-882, symbol Diode:PESD5V0L1UL
- added R10, R9: 220, symbol Device:R_US
- added R11: 47, symbol Device:R_US
- added R3, R4: 10k, symbol Device:R_US
- renumbered J3C to J3, J3P to J3P1, J4C to J4, J4P to J4P1, J5C to J5, J5P to J5P1, U5 to U2, U2 to U3
Connections:
- net 3.3V: now also R11.2, R3.1, R4.1; no longer C8.1, C9.1, J5.1 (Pin_1), U1.13 (VDDA)
- net GND: now also D1.2 (A), D2.2 (A), D3.2 (A)
- net at C12.1, U1.10 (PC2): now also R10.2, R4.2; no longer J4.1 (Pin_1)
- net at C11.1, U1.9 (PC1): now also R3.2, R9.2; no longer J3.1 (Pin_1)
- net at J5.2 (Pin_2), R8.1: now also D1.1 (K)
- new net: D3.1 (K), J4.1 (Pin_1), R10.1
- new net: D2.1 (K), J3.1 (Pin_1), R9.1
- new net VDDA: C8.1, C9.1, J5.1 (Pin_1), R11.1, U1.13 (VDDA)
Other:
- moved on the sheet: C12, J3, J4, J5, R7
